File: pcbs/swoopt-soldered/swoopt-soldered.kicad_sch (KiCad schematic)
At the start: 61 parts, among them J1 TRRS, SW1 MX, SW10 MX, SW11 MX, SW12 MX, SW13 MX, SW14 MX, SW15 MX, SW16 MX, SW17 MX, SW18 MX, SW2 MX, SW3 MX, SW4 MX, SW5 MX, SW6 MX, SW7 MX, SW8 MX, SW9 MX, U1 ProMicro

Commit message: updated footprints and traces. Also added Debora.
Parts:
- removed U1: ProMicro, swoop:ProMicro_jumpers, symbol swoop:ProMicro-kbd-corne-light-rescue
- added U1: ~, mcu:U_ProMicro_nRF52840_TH_Reversible, symbol inpulib:U_ProMicro_nRF52840
Connections:
- net GND: now also U1.23 (GND), U1.3 (GND), U1.4 (GND); no longer PSW1.2 (B)
- net VCC: now also U1.21 (VCC)
- net col0: now also U1.16 (B1/15)
- net col1: now also U1.17 (F7/A0)
- net col2: now also U1.18 (F6/A1)
- net col3: now also U1.19 (F5/A2)
- net col4: now also U1.20 (F4/A3)
- net data: now also U1.2 (RX1/D2)
- net eda: now also U1.11 (8/B4)
- net edb: now also U1.12 (9/B5)
- net led: now also U1.1 (TX0/D3)
- net reset: now also U1.22 (RST)
- net row0: now also U1.7 (4/D4)
- net row1: now also U1.8 (5/C6)
- net row2: now also U1.9 (6/D7)
- net row3: now also U1.10 (7/E6)
- net sda: now also U1.5 (2/D1/SDA)
- net sla: now also U1.6 (3/D0/SCL)
- net raw renamed bat+
- net bat+: now also U1.26 (BAT+)
- new net bat-: PSW1.2 (B), U1.25 (BAT-)
- no-connect marks 5 -> 6
Other:
- moved on the sheet: EN1, L1, L10, L11, L12, L13, L14, L15, L16, L17, L18, L2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

Commit message: work on the swoopiest - layout defined
Parts:
- added D19, D20, D21: 1N4148, swoop:D_SMD_TH, symbol Device:D_Small
- added L11, L17, L21: SK6812Mini-e, swoop:SK6812_Mini_E, symbol swoop:SK6812MINI-E
- added SW11, SW17, SW21: MX, switches:SW_Universal_TH_Reversible, symbol Switch:SW_Push
- D1, D10, D11, D12, D13, D14, D15, D16, D17, D18, D2, D3, D4, D5, D6, D7, D8, D9: value 1N4148W -> 1N4148
- SW1, SW10, SW2, SW3, SW4, SW5, SW6, SW7, SW8, SW9: footprint switches:SW_Universal_TH -> switches:SW_Universal_TH_Reversible
- SW12: renamed from SW11; footprint switches:SW_Universal_TH -> switches:SW_Universal_TH_Reversible
- SW13: renamed from SW12; footprint switches:SW_Universal_TH -> switches:SW_Universal_TH_Reversible
- SW14: renamed from SW13; footprint switches:SW_Universal_TH -> switches:SW_Universal_TH_Reversible
- SW15: renamed from SW14; footprint switches:SW_Universal_TH -> switches:SW_Universal_TH_Reversible
- SW16: renamed from SW15; footprint switches:SW_Universal_TH -> switches:SW_Universal_TH_Reversible
- SW18: renamed from SW16; footprint switches:SW_Universal_TH -> switches:SW_Universal_TH_Reversible
- SW19: renamed from SW17; footprint switches:SW_Universal_TH -> switches:SW_Universal_TH_Reversible
- SW20: renamed from SW18; footprint switches:SW_Universal_TH -> switches:SW_Universal_TH_Reversible
- renumbered L11 to L12, L12 to L13, L13 to L14, L14 to L15, L15 to L16, L16 to L18, L17 to L19, L18 to L20
Connections:
- net GND: now also L11.3 (VSS), L17.3 (VSS), L21.3 (VSS)
- net VCC: now also L11.1 (VDD), L17.1 (VDD), L21.1 (VDD)
- net er0: now also D18.2 (A); no longer D16.2 (A)
- net led: now also L11.4 (DIN); no longer L20.4 (DIN)
- net row1: now also D11.1 (K)
- net row2: now also D16.1 (K), D17.1 (K); no longer D11.1 (K)
- net row3: now also D19.1 (K), D20.1 (K), D21.1 (K); no longer D16.1 (K), D17.1 (K)
- net at SW12.2: now also D12.2 (A); no longer D11.2 (A)
- net at SW14.2: now also D14.2 (A); no longer D13.2 (A)
- net at SW20.2: now also D20.2 (A); no longer D18.2 (A)
- net at SW15.2: now also D15.2 (A); no longer D14.2 (A)
- net at D17.2 (A): now also SW17.2; no longer SW19.2
- net at SW16.2: now also D16.2 (A); no longer D15.2 (A)
- net at SW13.2: now also D13.2 (A); no longer D12.2 (A)
- net col5: now reaches U1.15 (B3/14)
- net col5: now also SW11.1, SW17.1, SW21.1
- new net: L11.2 (DOUT), L17.4 (DIN)
- new net: D21.2 (A), SW21.2
- new net: D19.2 (A), SW19.2
- new net: L20.4 (DIN), L21.2 (DOUT)
- new net: L17.2 (DOUT), L21.4 (DIN)
- new net: D11.2 (A), SW11.2
- no-connect marks 6 -> 5

Commit message: traces are complete, with second jack
Connections:
- net at L19.2 (DOUT): now also L18.4 (DIN); no longer L14.4 (DIN)
- net at L18.2 (DOUT): now also L14.4 (DIN)
- net at L1.2 (DOUT): no longer L18.4 (DIN)
Other:
- moved on the sheet: L18
Changed lines of the file:
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@@
 	)
 	(no_connect
-		(at 62.23 53.34)
+		(at 39.37 118.11)
 	)
 	(no_connect
-		(at 64.77 186.69)
+		(at 62.23 53.34)
 	)
 	(no_connect
@@
 	(wire
 		(pts
-			(xy 29.21 118.11) (xy 29.21 171.45)
-		)
-		(stroke
-			(width 0)
-			(type default)
-		)
-	)
-	(wire
-		(pts
 			(xy 92.71 143.51) (xy 92.71 161.29)
 		)
@@
 	(wire
 		(pts
-			(xy 39.37 133.35) (xy 39.37 135.89)
+			(xy 62.23 161.29) (xy 62.23 179.07)
 		)
 		(stroke
@@
 	(wire
 		(pts
-			(xy 62.23 27.94) (xy 67.31 27.94)
+			(xy 39.37 133.35) (xy 39.37 135.89)
 		)
 		(stroke
 			(width 0)
-			(type solid)
+			(type default)
 		)
 	)
 	(wire
 		(pts
-			(xy 74.93 168.91) (xy 69.85 168.91)
+			(xy 62.23 27.94) (xy 67.31 27.94)
 		)
 		(stroke
 			(width 0)
-			(type default)
+			(type solid)
 		)
 	)
@@
 	(wire
 		(pts
-			(xy 74.93 186.69) (xy 74.93 168.91)
-		)
-		(stroke
-			(width 0)
-			(type default)
-		)
-	)
-	(wire
-		(pts
 			(xy 123.19 143.51) (xy 123.19 161.29)
 		)
@@
 	(wire
 		(pts
-			(xy 39.37 118.11) (xy 29.21 118.11)
-		)
-		(stroke
-			(width 0)
-			(type default)
-		)
-	)
-	(wire
-		(pts
 			(xy 78.74 110.49) (xy 91.44 110.49)
 		)
@@
 	(wire
 		(pts
-			(xy 74.93 186.69) (xy 85.09 186.69)
+			(xy 118.11 48.26) (xy 125.73 48.26)
 		)
 		(stroke
 			(width 0)
-			(type default)
+			(type solid)
 		)
 	)
 	(wire
 		(pts
-			(xy 118.11 48.26) (xy 125.73 48.26)
+			(xy 77.47 125.73) (xy 77.47 143.51)
 		)
 		(stroke
 			(width 0)
-			(type solid)
+			(type default)
 		)
 	)
 	(wire
 		(pts
-			(xy 77.47 125.73) (xy 77.47 143.51)
+			(xy 100.33 151.13) (xy 100.33 153.67)
 		)
 		(stroke
@@
 	(wire
 		(pts
-			(xy 100.33 151.13) (xy 100.33 153.67)
+			(xy 69.85 168.91) (xy 69.85 171.45)
 		)
 		(stroke
@@
 	(wire
 		(pts
-			(xy 78.74 90.17) (xy 91.44 90.17)
+			(xy 69.85 186.69) (xy 85.09 186.69)
 		)
 		(stroke
@@
 	(wire
 		(pts
-			(xy 39.37 151.13) (xy 39.37 153.67)
+			(xy 78.74 90.17) (xy 91.44 90.17)
 		)
 		(stroke
@@
 	(wire
 		(pts
-			(xy 29.21 171.45) (xy 64.77 171.45)
+			(xy 39.37 151.13) (xy 39.37 153.67)
 		)
 		(stroke
@@
 	)
 	(symbol
-		(lib_name "VCC_1")
-		(lib_id "power:VCC")
-		(at 72.39 179.07 0)
-		(unit 1)
-		(exclude_from_sim no)
-		(in_bom yes)
-		(on_board yes)
-		(dnp no)
-		(fields_autoplaced yes)
-		(property "Reference" "#PWR018"
-			(at 72.39 182.88 0)
-			(effects
-				(font
-					(size 1.27 1.27)
-				)
-				(hide yes)
-			)
-		)
-		(property "Value" "VCC"
-			(at 72.39 173.99 0)
-			(effects
-				(font
-					(size 1.27 1.27)
-				)
-			)
-		)
-		(property "Footprint" ""
-			(at 72.39 179.07 0)
-			(effects
-				(font
-					(size 1.27 1.27)
-				)
-				(hide yes)
-			)
-		)
-		(property "Datasheet" ""
-			(at 72.39 179.07 0)
-			(effects
-				(font
-					(size 1.27 1.27)
-				)
-				(hide yes)
-			)
-		)
-		(property "Description" "Power symbol creates a global label with name \"VCC\""
-			(at 72.39 179.07 0)
-			(effects
-				(font
-					(size 1.27 1.27)
-				)
-				(hide yes)
-			)
-		)
-		(pin "1"
-		)
-		(instances
-			(project "swoopt-soldered"
-				(path "/471b6803-5d15-4f73-aeb4-3a263e2bc423"
-					(reference "#PWR018")
-					(unit 1)
-				)
-			)
-		)
-	)
-	(symbol
 		(lib_name "D_Small_1")
 		(lib_id "Device:D_Small")
@@
 	)
 	(symbol
-		(lib_name "GND_1")
-		(lib_id "power:GND")
-		(at 57.15 179.07 0)
-		(unit 1)
-		(exclude_from_sim no)
-		(in_bom yes)
-		(on_board yes)
-		(dnp no)
-		(fields_autoplaced yes)
-		(property "Reference" "#PWR017"
-			(at 57.15 185.42 0)
-			(effects
-				(font
-					(size 1.27 1.27)
-				)
-				(hide yes)
-			)
-		)
-		(property "Value" "GND"
-			(at 57.15 184.15 0)
-			(effects
-				(font
-					(size 1.27 1.27)
-				)
-			)
-		)
-		(property "Footprint" ""
-			(at 57.15 179.07 0)
-			(effects
-				(font
-					(size 1.27 1.27)
-				)
-				(hide yes)
-			)
-		)
-		(property "Datasheet" ""
-			(at 57.15 179.07 0)
-			(effects
-				(font
-					(size 1.27 1.27)
-				)
-				(hide yes)
-			)
-		)
-		(property "Description" "Power symbol creates a global label with name \"GND\" , ground"
-			(at 57.15 179.07 0)
-			(effects
-				(font
-					(size 1.27 1.27)
-				)
-				(hide yes)
-			)
-		)
-		(pin "1"
-		)
-		(instances
-			(project "swoopt-soldered"
-				(path "/471b6803-5d15-4f73-aeb4-3a263e2bc423"
-					(reference "#PWR017")
-					(unit 1)
-				)
-			)
-		)
-	)
-	(symbol
 		(lib_id "inpulib:U_ProMicro_nRF52840")
 		(at 44.45 39.37 0)
@@
 	(symbol
 		(lib_id "swoop:SK6812MINI-E")
-		(at 64.77 179.07 270)
+		(at 69.85 179.07 90)
 		(unit 1)
 		(exclude_from_sim no)
@@
 		(dnp no)
 		(property "Reference" "L18"
-			(at 60.325 175.26 90)
+			(at 74.295 182.88 90)
 			(effects
 				(font
@@
 		)
 		(property "Value" "SK6812Mini-e"
-			(at 67.945 184.785 90)
+			(at 66.675 173.355 90)
 			(effects
 				(font
@@
 		)
 		(property "Footprint" "swoop:SK6812_Mini_E"
-			(at 64.77 179.07 0)
+			(at 69.85 179.07 0)
 			(effects
 				(font
@@
 		)
 		(property "Datasheet" ""
-			(at 64.77 179.07 0)
+			(at 69.85 179.07 0)
 			(effects
 				(font
@@
 		)
 		(property "Description" ""
-			(at 64.77 179.07 0)
+			(at 69.85 179.07 0)
 			(effects
 				(font
@@
 		)
 		(property "JLCPCB BOM" "0"
-			(at 64.77 179.07 0)
+			(at 69.85 179.07 0)
 			(effects
 				(font

Commit message: added underglow leds
Parts:
- added EN2, EN3: RotaryEncoder_Switch, swoop:RotaryEncoder, symbol Device:RotaryEncoder_Switch
- added L22, L23, L24, L25: SK6812Mini-e, diode:LED_SK6812MINI__3.5x3.5mm_reversible, symbol swoop:SK6812MINI-E
Connections:
- net GND: now also EN2.C, EN3.C, L22.3 (VSS), L23.3 (VSS), L24.3 (VSS), L25.3 (VSS)
- net VCC: now also L22.1 (VDD), L23.1 (VDD), L24.1 (VDD), L25.1 (VDD)
- net col5: now also EN2.S1, EN3.S1
- net eda: now also EN2.A, EN3.A
- net edb: now also EN2.B, EN3.B
- net er2: now reaches D17.2 (A), SW17.2
- net er2: now also EN3.S2
- net er1: now reaches D11.2 (A), SW11.2
- net er1: now also EN2.S2
- net at L1.2 (DOUT): now also L22.4 (DIN)
- new net: L23.2 (DOUT), L24.4 (DIN)
- new net: L22.2 (DOUT), L23.4 (DIN)
- new net: L24.2 (DOUT), L25.4 (DIN)
Other:
- moved on the sheet: L1, L10, L11, L12, L13, L14, L15, L16, L17, L18, L19, L2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
