File: pcbs/swoopt-soldered/swoopt-soldered.kicad_pcb (KiCad board)
At the start: 2 copper layers, 137.6 x 110.1 mm, 85 parts, among them J1 TRRS, SW1 MX, SW10 MX, SW11 MX, SW12 MX, SW13 MX, SW14 MX, SW15 MX, SW16 MX, SW17 MX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

Commit message: pulled pinky column 2mm down
Parts:
- added REF**: MountingHole_2.2mm_M2_ISO7380_Pad, MountingHole:MountingHole_2.2mm_M2_ISO7380_Pad, F.Cu at (184.8, 94.0)
- added REF**: MountingHole_2.2mm_M2_ISO7380_Pad, MountingHole:MountingHole_2.2mm_M2_ISO7380_Pad, F.Cu at (213.0, 103.5)
- moved REF** 8.72 mm to (209.2, 59.5)
- moved D1 2.25 mm to (94.0, 83.5)
- moved D12 2.25 mm to (94.0, 121.5)
- moved D6 2.25 mm to (94.0, 102.5)
- moved L1 2.25 mm to (94.0, 70.3)
- moved L12 2.25 mm to (94.0, 108.3)
- moved L6 2.25 mm to (94.0, 89.3)
- moved SW1 2.25 mm to (94.0, 75.2)
- moved SW12 2.25 mm to (94.0, 113.2)
- moved SW6 2.25 mm to (94.0, 94.2)
- moved RSW1 2.25 mm to (97.0, 60.2)
- moved REF** 2.00 mm to (94.0, 65.0)
Routing:
- net row1: track 182.7 -> 188.3 mm, vias 4 -> 6
- net VCC: track 635.3 -> 638.6 mm, vias 10 -> 11
- net Net-(L1-DIN): track 27.9 -> 30.3 mm
- net Net-(L1-DOUT): track 20.0 -> 17.8 mm
- net reset: track 127.5 -> 125.3 mm
- net row0: track 117.0 -> 119.2 mm
- net Net-(L12-DIN): track 51.8 -> 50.6 mm
- net col0: track 166.3 -> 165.3 mm, vias 6 -> 5
- net row2: track 179.4 -> 180.3 mm
Other:
- outline, holes or cut-outs redrawn

Commit message: added tenting puck
Parts:
- removed the REF** at (209.2, 59.5)
- removed the REF** at (193.5, 126.5)
- removed the REF** at (132.8, 105.0)
- removed the REF** at (184.8, 94.0)
- removed the REF** at (141.5, 52.2)
- removed the REF** at (213.0, 103.5)
- removed the REF** at (94.0, 65.0)
- added ?: , , F.Cu at (160.5, 63.0)
- added REF**: Tenting Puck, no hole, tenting_puck-main:TentingPuck_NoHole, F.Cu at (141.5, 88.5)
- added REF**: MountingHole_5.3mm_M5_ISO14580_Pad, MountingHole:MountingHole_5.3mm_M5_ISO14580_Pad, F.Cu at (89.5, 56.5)
- moved RSW1 2.37 mm to (99.2, 61.0), turned to 90 degrees
Connections:
- REF** pad 1: (no net) -> GND (x2)
Routing:
- net col1: track 141.9 -> 149.1 mm
- net VCC: track 638.6 -> 645.8 mm, vias 11 -> 10
- net GND: track 715.9 -> 710.4 mm
- net col3: track 125.1 -> 119.8 mm
- net Net-(L18-DIN): track 36.7 -> 41.0 mm
- net edb: track 140.2 -> 143.8 mm
- net eda: track 143.1 -> 146.8 mm
- net col0: track 165.3 -> 168.6 mm
- net reset: track 125.3 -> 122.3 mm
- net unconnected-(L25-DOUT-Pad2)_1: track 0.00 -> 2.61 mm
- net Net-(L24-DOUT): track 78.3 -> 76.3 mm
- net row1: track 188.3 -> 190.3 mm
- net Net-(L22-DOUT): track 76.9 -> 78.8 mm
- net row2: track 180.3 -> 181.6 mm
- net col2: track 139.5 -> 138.3 mm, vias 7 -> 9
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